File: starbie/starbie.kicad_sch (KiCad schematic)
At the start: 7 parts, among them J1 Conn_01x04_Pin, J2 Conn_01x08_Pin, SW1 SW_Push, SW2 SW_Push, U1 XIAO-ESP32-C3-SMD, U2 DHT11

Commit message: updated schematic and pcb to use SDA and SCL correct way round
Connections:
- net SCL: now also U1.6 (D5); no longer U1.5 (D4)
- net SDA: now also U1.5 (D4); no longer U1.6 (D5)
Changed lines of the file:
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@@
 		)
 	)
-	(label "SDA"
+	(label "SCL"
 		(at 38.1 77.47 180)
 		(effects
@@
 		)
 	)
-	(label "SCL"
+	(label "SDA"
 		(at 38.1 73.66 180)
 		(effects
